File: blackMD_mother.kicad_sch (KiCad schematic)
At the start: 14 parts, among them J1 MD_Socket1, J10 I2C_OUT, J11 PWR_IN, J2 MD_Socket2, J3 MD_Socket3, J4 MD_Socket4, J5 XT_Motor1, J6 XT_Motor2, J7 XT_Motor3, J8 XT_Motor4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

Commit message: swap MotorA & MotorB
Parts:
- I2C1: renamed from J9; value I2C_IN -> S04B
- I2C2: renamed from J10; value I2C_OUT -> S04B
- MD1: renamed from J1; value MD_Socket1 -> XG4A-5071
- MD2: renamed from J2; value MD_Socket2 -> XG4A-5071
- MD3: renamed from J3; value MD_Socket3 -> XG4A-5071
- MD4: renamed from J4; value MD_Socket4 -> XG4A-5071
- MotorOUT1: renamed from J5; value XT_Motor1 -> XT60
- MotorOUT2: renamed from J6; value XT_Motor2 -> XT60
- MotorOUT3: renamed from J7; value XT_Motor3 -> XT60
- MotorOUT4: renamed from J8; value XT_Motor4 -> XT60
Connections:
- net Motor_1A: now also MotorOUT1.2 (Pin_2); no longer MotorOUT1.1 (Pin_1)
- net Motor_1B: now also MotorOUT1.1 (Pin_1); no longer MotorOUT1.2 (Pin_2)
- net Motor_2A: now also MotorOUT2.2 (Pin_2); no longer MotorOUT2.1 (Pin_1)
- net Motor_2B: now also MotorOUT2.1 (Pin_1); no longer MotorOUT2.2 (Pin_2)
- net Motor_3A: now also MotorOUT3.2 (Pin_2); no longer MotorOUT3.1 (Pin_1)
- net Motor_3B: now also MotorOUT3.1 (Pin_1); no longer MotorOUT3.2 (Pin_2)
- net Motor_4A: now also MotorOUT4.2 (Pin_2); no longer MotorOUT4.1 (Pin_1)
- net Motor_4B: now also MotorOUT4.1 (Pin_1); no longer MotorOUT4.2 (Pin_2)
Other:
- moved on the sheet: MotorOUT1, MotorOUT2, MotorOUT3, MotorOUT4

Commit message: update silk
Parts:
- MotorOUT1, MotorOUT2, MotorOUT3, MotorOUT4: value XT60 -> XT60_F
- PowerIn1: renamed from J11; value PWR_IN -> XT60_M
Changed lines of the file:
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@@
       (effects (font (size 1.27 1.27)))
     )
-    (property "Value" "XT60" (at 198.755 54.61 0)
+    (property "Value" "XT60_F" (at 198.755 54.61 0)
       (effects (font (size 1.27 1.27)))
     )
@@
       (effects (font (size 1.27 1.27)))
     )
-    (property "Value" "XT60" (at 117.475 54.61 0)
+    (property "Value" "XT60_F" (at 117.475 54.61 0)
       (effects (font (size 1.27 1.27)))
     )
@@
       (effects (font (size 1.27 1.27)))
     )
-    (property "Value" "XT60" (at 159.385 54.61 0)
+    (property "Value" "XT60_F" (at 159.385 54.61 0)
       (effects (font (size 1.27 1.27)))
     )
@@
   (symbol (lib_id "Connector:Conn_01x02_Socket") (at 215.9 104.14 180) (unit 1)
     (in_bom yes) (on_board yes) (dnp no) (fields_autoplaced)
-    (property "Reference" "J11" (at 216.535 96.52 0)
-      (effects (font (size 1.27 1.27)))
-    )
-    (property "Value" "PWR_IN" (at 216.535 99.06 0)
+    (property "Reference" "PowerIn1" (at 216.535 96.52 0)
+      (effects (font (size 1.27 1.27)))
+    )
+    (property "Value" "XT60_M" (at 216.535 99.06 0)
       (effects (font (size 1.27 1.27)))
     )
@@
       (project "blackMD_mother"
         (path "/ea97f4a9-09a5-44cb-b831-5400ff5dc24b"
-          (reference "J11") (unit 1)
+          (reference "PowerIn1") (unit 1)
         )
       )
@@
       (effects (font (size 1.27 1.27)))
     )
-    (property "Value" "XT60" (at 75.565 54.61 0)
-      (effects (font (size 1.27 1.27)))
-    )
+    (property "Value" "XT60_F" (at 75.565 54.61 0)
+      (effects (font (size 1.27 1.27)))
+    )
